Commit message: new laser mount

File: src/wrock_husky_description/urdf/husky.urdf.xacro (robot description, xacro)
@@ -211,6 +211,6 @@
     </link>
     <joint name="cube_joint" type="continuous">
-		<origin xyz="-0.07 0 0" rpy="0 0 0" />
-	  <axis xyz="-1 0 0" />
+		<origin xyz="0 0 -0.07" rpy="0 0 0" />
+	  <axis xyz="0 0 -1 " />
         <parent link="fixed_cube_5"/>
         <child link="cube_5" />
@@ -222,5 +222,5 @@
         <origin xyz="0 0 0" rpy="0 0 0" />
         <geometry>
-          <!-- Origin of this mesh is the base of the bracket. -->
+          <!-- Origin of this mesh is the base of the bracket. -${M_PI/2}-->
           <mesh filename="package://wrock_husky_description/meshes/sick_lms1xx.dae" />
         </geometry>
@@ -229,5 +229,5 @@
     </link>
     <joint name="laser_mount_joint" type="fixed">
-      <origin xyz="-.0285 -0.1 0" rpy="0 0 -${M_PI/2}" />
+      <origin xyz="-.0285 -0.1 0" rpy="${M_PI/2} 0 -${M_PI/2}" />
       <parent link="cube_5" />
       <child link="laser" />

Commit message: updating

File: src/wrock_husky_description/urdf/husky.urdf.xacro (robot description, xacro)
@@ -163,5 +163,5 @@
     </link>
     <joint name="base_cube_joint" type="fixed">
-		<origin xyz="0.265 .2005 ${0.445 + 0.35550000/2 - 0.03282508}" rpy="${M_PI} ${M_PI/2} 0" />
+		<origin xyz="0.165 .2005 ${0.445 + 0.35550000/2 - 0.03282508}" rpy="${M_PI} ${M_PI/2} 0" />
         <parent link="base_footprint"/>
         <child link="angle_connector" />
