Commit message: fixed husky bugs

File: src/wrock_husky_description/urdf/base.urdf.xacro (robot description, xacro)
@@ -235,5 +235,5 @@
         </visual>
     </link>
-    <joint name="cube_5_joint" type="continuous">
+    <joint name="cube_joint" type="continuous">
 		<origin xyz="-0.07 0 0" rpy="0 0 0" />
 	  <axis xyz="-1 0 0" />

File: src/wrock_husky_description/urdf/husky.urdf.xacro (robot description, xacro)
@@ -210,5 +210,5 @@
         </visual>
     </link>
-    <joint name="cube_5_joint" type="continuous">
+    <joint name="cube_joint" type="continuous">
 		<origin xyz="-0.07 0 0" rpy="0 0 0" />
 	  <axis xyz="-1 0 0" />

Commit message: arm movement

File: src/wrock_husky_description/urdf/base.urdf.xacro (robot description, xacro)
@@ -188,5 +188,5 @@
     </link>
     <joint name="base_cube_joint" type="fixed">
-		<origin xyz="0.265 .2005 ${0.345 + wheel_x_size/2 - base_z_origin_to_wheel_origin}" rpy="${M_PI} ${M_PI/2} 0" />
+		<origin xyz="0.265 .2005 ${0.445 + wheel_x_size/2 - base_z_origin_to_wheel_origin}" rpy="${M_PI} ${M_PI/2} 0" />
         <parent link="base_footprint"/>
         <child link="angle_connector" />
@@ -416,5 +416,5 @@
   </joint>
       <joint name="Arm_Mount" type="fixed">
-      <origin xyz="0 0 ${.3 + wheel_x_size/2 - base_z_origin_to_wheel_origin}" rpy="0 0 0" />
+      <origin xyz="1 -.20 ${.3 + wheel_x_size/2 - base_z_origin_to_wheel_origin}" rpy="0 0 ${M_PI}" />
       <parent link="base_footprint" />
       <child link="BASE" />

File: src/wrock_husky_description/urdf/husky.urdf.xacro (robot description, xacro)
@@ -163,5 +163,5 @@
     </link>
     <joint name="base_cube_joint" type="fixed">
-		<origin xyz="0.265 .2005 ${0.345 + 0.35550000/2 - 0.03282508}" rpy="${M_PI} ${M_PI/2} 0" />
+		<origin xyz="0.265 .2005 ${0.445 + 0.35550000/2 - 0.03282508}" rpy="${M_PI} ${M_PI/2} 0" />
         <parent link="base_footprint"/>
         <child link="angle_connector" />
@@ -391,5 +391,5 @@
   </joint>
       <joint name="Arm_Mount" type="fixed">
-      <origin xyz="0 0 ${.3 + 0.35550000/2 - 0.03282508}" rpy="0 0 0" />
+      <origin xyz=".156971 -.096013 .405369" rpy="0 0 ${M_PI}" />
       <parent link="base_footprint" />
       <child link="BASE" />

Commit message: march update

File: src/wrock_husky_description/urdf/base.urdf.xacro (robot description, xacro)
@@ -188,5 +188,5 @@
     </link>
     <joint name="base_cube_joint" type="fixed">
-		<origin xyz="0.265 .2005 ${0.445 + wheel_x_size/2 - base_z_origin_to_wheel_origin}" rpy="${M_PI} ${M_PI/2} 0" />
+		<origin xyz=".195262 .31089 .49343" rpy="0 0 0" />
         <parent link="base_footprint"/>
         <child link="angle_connector" />

File: src/wrock_husky_description/urdf/husky.urdf.xacro (robot description, xacro)
@@ -155,5 +155,5 @@
             <origin xyz="0 0 0" rpy="0 0 0" />
             <geometry>
-                <mesh filename="package://wrock_husky_description/meshes/cubefinal.stl" />
+                <mesh filename="file:///home/mike/catkin_ws/src/wrock_husky_description/meshes/Bracket.stl" scale="0.001 0.001 0.001"/>
             </geometry>
             <material name="DarkPCubeGrey" >
@@ -163,5 +163,5 @@
     </link>
     <joint name="base_cube_joint" type="fixed">
-		<origin xyz="0.165 .2005 ${0.445 + 0.35550000/2 - 0.03282508}" rpy="${M_PI} ${M_PI/2} 0" />
+		<origin xyz="${.31089+.094967} ${.195262 - .047625} ${.50343-.247016}" rpy="0.698132 0 ${M_PI/2}" />
         <parent link="base_footprint"/>
         <child link="angle_connector" />
@@ -177,5 +177,5 @@
         </inertial>
         <visual>
-            <origin xyz="0 0 0" rpy="0 0 0" />
+            <origin xyz="-.035 -.035 -.035" rpy="0 0 0" />
             <geometry>
                 <box size="0.07 0.07 0.07" />
@@ -187,5 +187,5 @@
     </link>
     <joint name="fixed_cube_5_joint" type="fixed">
-		<origin xyz="0.035 0.035 -0.035" rpy="0 0 ${-M_PI/2}" />
+		<origin xyz="${.047625} ${.231527766824} ${.128181623232}" rpy="${-.698132} 0 0" />
         <parent link="angle_connector"/>
         <child link="fixed_cube_5" />
@@ -211,5 +211,5 @@
     </link>
     <joint name="cube_joint" type="continuous">
-		<origin xyz="0 0 -0.07" rpy="0 0 0" />
+		<origin xyz="-.035 -.105 -.035" rpy="-${M_PI/2} 0 0" />
 	  <axis xyz="0 0 -1 " />
         <parent link="fixed_cube_5"/>
@@ -220,14 +220,17 @@
     <link name="laser">
       <visual>
-        <origin xyz="0 0 0" rpy="0 0 0" />
+        <origin xyz="0 0 0" rpy="0 0 ${M_PI/2}" />
         <geometry>
           <!-- Origin of this mesh is the base of the bracket. -${M_PI/2}-->
-          <mesh filename="package://wrock_husky_description/meshes/sick_lms1xx.dae" />
+          <mesh filename="file:///home/mike/catkin_ws/src/wrock_husky_description/meshes/laser.stl" scale = "0.001 0.001 0.001"/>
         </geometry>
-        <material name="dark_grey" />
+            <material name="white">
+        <color rgba="1 1 1 1"/>
+      </material>
       </visual>
     </link>
     <joint name="laser_mount_joint" type="fixed">
-      <origin xyz="-.0285 -0.1 0" rpy="${M_PI/2} 0 -${M_PI/2}" />
+      <!--<origin xyz="${.019663 - .035} ${-.035 - .05974} -.027623" rpy="${M_PI/2} 0 ${-M_PI/2}" />-->
+<origin xyz="${.019663 -.027623} ${-.035 - .05974} -.027623" rpy="${M_PI/2} 0 ${-M_PI/2}" />
       <parent link="cube_5" />
       <child link="laser" />
